Commit message: a lot of small changes that make the robot actually walk irl git log

File: data/idefX/idefX.urdf (robot description, URDF)
Before this commit: robot idefX, 26 links, 25 joints
Joints:
- joint BL_clavicle_joint: origin xyz=-0.225 0.075 -0.0 rpy=0 0 0 -> xyz=-0.225 0.0575 -0.0 rpy=0 0 0
- joint BL_first_motor_joint: origin xyz=-0.15250000000000002 0.075 0.0 rpy=0 0 0 -> xyz=-0.15250000000000002 0.0575 0.0 rpy=0 0 0
- joint BR_clavicle_joint: origin xyz=-0.225 -0.075 -0.0 rpy=0 0 0 -> xyz=-0.225 -0.0575 -0.0 rpy=0 0 0
- joint BR_first_motor_joint: origin xyz=-0.15250000000000002 -0.075 0.0 rpy=0 0 0 -> xyz=-0.15250000000000002 -0.0575 0.0 rpy=0 0 0
- joint FL_clavicle_joint: origin xyz=0.225 0.075 -0.0 rpy=0 0 0 -> xyz=0.225 0.0575 -0.0 rpy=0 0 0
- joint FL_first_motor_joint: origin xyz=0.15250000000000002 0.075 0.0 rpy=0 0 0 -> xyz=0.15250000000000002 0.0575 0.0 rpy=0 0 0
- joint FR_clavicle_joint: origin xyz=0.225 -0.075 -0.0 rpy=0 0 0 -> xyz=0.225 -0.0575 -0.0 rpy=0 0 0
- joint FR_first_motor_joint: origin xyz=0.15250000000000002 -0.075 0.0 rpy=0 0 0 -> xyz=0.15250000000000002 -0.0575 0.0 rpy=0 0 0
